Commit message: Not so sneaky if you break simulation.launch

File: urdf/ar_mark.urdf (robot description, URDF)
Before this commit: robot ar_mark, 1 links, 0 joints
Links:
- link ar_link: mass 1 -> 0.1; geometry collision box size=0.2 0.2 0.2; visual mesh filename=package://kvaradrive/urdf/artag.dae scale=1 1 1

Commit message: keeps publishing old goal in map frame if marker is lost; changed collisions of marker

File: urdf/ar_mark.urdf (robot description, URDF)
Before this commit: robot ar_mark, 1 links, 0 joints
Links:
- link ar_link: geometry collision box size=0.05 0.05 0.1; visual mesh filename=package://kvaradrive/urdf/artag.dae scale=1 1 1
