Commit message: Resolved file name conflicts

File: urdf/lidar_gazebo_macro.xacro (robot description, xacro)
@@ -1,5 +1,5 @@
 <?xml version="1.0"?>
 <robot name="lidar_gazebo_macro" xmlns:xacro="http://www.ros.org/wiki/xacro">
-  <!--xacro:include filename="$(find mr_description)/urdf/utility_macro.xacro" /-->
+  <!--xacro:include filename="$(find kvaradrive)/urdf/utility_macro.xacro" /-->
   <xacro:macro name="lidar_gazebo_sensor" params="parent" >
     <link name="laser_frame">
@@ -12,5 +12,5 @@
       <visual>
         <geometry>
-          <mesh filename="package://mr_description/meshes/lidar.stl" scale="0.001 0.001 0.001 "/>
+          <mesh filename="package://kvaradrive/meshes/lidar.stl" scale="0.001 0.001 0.001 "/>
         </geometry>
         <material name="White"/>

File: urdf/mr.xacro (robot description, xacro)
@@ -1,5 +1,5 @@
 <?xml version="1.0"?>
 <robot name="mobile_robot" xmlns:xacro="http://ros.org/wiki/xacro">
-  <xacro:include filename="$(find mr_description)/urdf/mr_base_macro.xacro" />
+  <xacro:include filename="$(find kvaradrive)/urdf/mr_base_macro.xacro" />
   <!-- Diff Drive Robot Base  -->
   <xacro:mr_base />

File: urdf/mr_base_macro.xacro (robot description, xacro)
@@ -1,5 +1,5 @@
 <?xml version="1.0"?>
 <robot name="mr_base_macro" xmlns:xacro="http://www.ros.org/wiki/xacro">
-  <xacro:include filename="$(find mr_description)/urdf/utility_macro.xacro" />
+  <xacro:include filename="$(find kvaradrive)/urdf/utility_macro.xacro" />
   <!-- Base properties -->
 	<xacro:property name="base_height" value="0.180" />
@@ -23,5 +23,5 @@
       <visual>
         <geometry>
-          <mesh filename="package://mr_description/meshes/mr_body.stl" scale="0.001 0.001 0.001 "/>
+          <mesh filename="package://kvaradrive/meshes/mr_body.stl" scale="0.001 0.001 0.001 "/>
         </geometry>
         <material name="White"/>
@@ -44,5 +44,5 @@
       <visual>
         <geometry>
-          <mesh filename="package://mr_description/meshes/mr_wheel.stl" scale="0.001 0.001 0.001 "/>
+          <mesh filename="package://kvaradrive/meshes/mr_wheel.stl" scale="0.001 0.001 0.001 "/>
         </geometry>
         <material name="Black"/>
@@ -51,5 +51,5 @@
       <collision>
         <geometry>
-          <mesh filename="package://mr_description/meshes/mr_wheel.stl" scale="0.001 0.001 0.001 "/>
+          <mesh filename="package://kvaradrive/meshes/mr_wheel.stl" scale="0.001 0.001 0.001 "/>
         </geometry>
         <origin rpy="0 0 0" xyz="0 0 0"/>
@@ -66,5 +66,5 @@
       <visual>
         <geometry>
-          <mesh filename="package://mr_description/meshes/mr_wheel.stl" scale="0.001 0.001 0.001 "/>
+          <mesh filename="package://kvaradrive/meshes/mr_wheel.stl" scale="0.001 0.001 0.001 "/>
         </geometry>
         <material name="Black"/>
@@ -73,5 +73,5 @@
       <collision>
         <geometry>
-          <mesh filename="package://mr_description/meshes/mr_wheel.stl" scale="0.001 0.001 0.001 "/>
+          <mesh filename="package://kvaradrive/meshes/mr_wheel.stl" scale="0.001 0.001 0.001 "/>
         </geometry>
         <origin rpy="0 0 0" xyz="0 0 0"/>

Commit message: lidar sensor corrections

File: urdf/lidar_gazebo_macro.xacro (robot description, xacro)
@@ -31,5 +31,5 @@
     <gazebo reference="laser_frame">
       <sensor type="ray" name="head_hokuyo_sensor">
-        <pose>0 0 0 0 0 0</pose>
+        <pose>0 0 0.38 0 0 0</pose>
         <visualize>true</visualize>
         <update_rate>40</update_rate>

File: urdf/mr.xacro (robot description, xacro)
@@ -2,7 +2,5 @@
 <robot name="mobile_robot" xmlns:xacro="http://ros.org/wiki/xacro">
   <xacro:include filename="$(find kvaradrive)/urdf/mr_base_macro.xacro" />
-  <xacro:include filename="$(find kvaradrive)/urdf/lidar_gazebo_macro.xacro" />
   <!-- Diff Drive Robot Base  -->
   <xacro:mr_base />
-  <xacro:lidar_gazebo_sensor parent="base_link" />
 </robot>

File: urdf/mr_base_macro.xacro (robot description, xacro)
@@ -127,4 +127,67 @@
       </actuator>
     </transmission>
+    <!--Lidar sensor -->
+ <link name="laser_frame">
+      <inertial>
+          <inertia ixx="1.0" ixy="0.0" ixz="0.0" iyy="1.0" iyz="0.0" izz="1.0"/>
+        <mass value="0.1" />
+        <origin xyz="0 0 0" />
+        <cylinder_inertia  m="0.1" r="0.037" h="0.04" />
+      </inertial>
+      <visual>
+        <geometry>
+          <mesh filename="package://kvaradrive/meshes/lidar.stl" scale="0.001 0.001 0.001 "/>
+        </geometry>
+        <material name="White"/>
+        <origin rpy="0 0 ${-M_PI_2}" xyz="0.0 0.0 -0.031"/>
+      </visual>
+      <collision>
+        <origin xyz="0 0 0" rpy="0 0 0 " />
+        <geometry>
+          <cylinder length="0.04" radius="0.037" />
+        </geometry>
+        <origin rpy="0 0 0" xyz="0.0 0.0 -0.031"/>
+      </collision>
+    </link>
+    <joint name="laser_joint" type="fixed">
+      <parent link="base_link"/>
+      <child link="laser_frame"/>
+      <origin rpy="0 0 0" xyz="0.0 0.0 0.155"/>
+    </joint>
+    <gazebo reference="laser_frame">
+      <sensor type="ray" name="head_hokuyo_sensor">
+        <pose>0 0 0 0 0 0</pose>
+        <visualize>true</visualize>
+        <update_rate>40</update_rate>
+        <ray>
+            <scan>
+              <horizontal>
+                <samples>720</samples>
+                <resolution>1</resolution>
+                <min_angle>-${M_PI} </min_angle>
+                <max_angle>${M_PI} </max_angle>
+              </horizontal>
+            </scan>
+            <range>
+              <min>0.8</min>
+              <max>30.0</max>
+              <resolution>0.01</resolution>
+            </range>
+            <noise>
+              <type>gaussian</type>
+              <!-- Noise parameters based on published spec for Hokuyo laser
+                    achieving "+-30mm" accuracy at range < 10m.  A mean of 0.0m and
+                    stddev of 0.01m will put 99.7% of samples within 0.03m of the true
+                    reading. -->
+              <mean>0.0</mean>
+              <stddev>0.01</stddev>
+            </noise>
+        </ray>
+        <plugin name="gazebo_ros_head_hokuyo_controller" filename="libgazebo_ros_laser.so">
+            <topicName>/laser/scan</topicName>
+            <frameName>laser_frame</frameName>
+        </plugin>
+      </sensor>
+    </gazebo>
     <!-- Differential drive controller  -->
   <gazebo>

Commit message: added lidar and camera to hardware

File: urdf/lidar_gazebo_macro.xacro (robot description, xacro)
@@ -2,5 +2,5 @@
 <robot name="lidar_gazebo_macro" xmlns:xacro="http://www.ros.org/wiki/xacro">
   <xacro:macro name="lidar_gazebo_sensor" params="parent" >
-    <link name="laser_frame">
+    <link name="laser">
       <inertial>
           <inertia ixx="1.0" ixy="0.0" ixz="0.0" iyy="1.0" iyz="0.0" izz="1.0"/>
@@ -26,8 +26,8 @@
     <joint name="laser_joint" type="fixed">
       <parent link="${parent}"/>
-      <child link="laser_frame"/>
+      <child link="laser"/>
       <origin rpy="0 0 0" xyz="0.0 0.0 0.031"/>
     </joint>
-    <gazebo reference="laser_frame">
+    <gazebo reference="laser">
       <sensor type="ray" name="head_hokuyo_sensor">
         <pose>0 0 0.38 0 0 0</pose>
@@ -60,5 +60,5 @@
         <plugin name="gazebo_ros_head_hokuyo_controller" filename="libgazebo_ros_laser.so">
             <topicName>/laser/scan</topicName>
-            <frameName>laser_frame</frameName>
+            <frameName>laser</frameName>
         </plugin>
       </sensor>

File: urdf/mr_base_macro.xacro (robot description, xacro)
@@ -128,5 +128,5 @@
     </transmission>
     <!--Lidar sensor -->
- <link name="laser_frame">
+ <link name="laser">
       <inertial>
           <inertia ixx="1.0" ixy="0.0" ixz="0.0" iyy="1.0" iyz="0.0" izz="1.0"/>
@@ -152,8 +152,8 @@
     <joint name="laser_joint" type="fixed">
       <parent link="base_link"/>
-      <child link="laser_frame"/>
+      <child link="laser"/>
       <origin rpy="0 0 0" xyz="0.0 0.0 0.155"/>
     </joint>
-    <gazebo reference="laser_frame">
+    <gazebo reference="laser">
       <sensor type="ray" name="head_hokuyo_sensor">
         <pose>0 0 0 0 0 0</pose>
@@ -186,5 +186,5 @@
         <plugin name="gazebo_ros_head_hokuyo_controller" filename="libgazebo_ros_laser.so">
             <topicName>/laser/scan</topicName>
-            <frameName>laser_frame</frameName>
+            <frameName>laser</frameName>
         </plugin>
       </sensor>
