Commit message: Transmission added but not actuated yet

File: urdf/mr_base_macro.xacro (robot description, xacro)
@@ -106,4 +106,24 @@
       <joint_properties damping="0.5" friction="0.01"/>
     </joint>
+    <transmission name="left_wheel_tran">
+      <type>transmission_interface/SimpleTransmission</type>
+      <joint name="left_wheel_joint">
+	<hardwareInterface>EffortJointInterface</hardwareInterface>
+      </joint>
+      <actuator name="left_wheel_motor">
+	<hardwareInterface>EffortJointInterface</hardwareInterface>
+	<mechanicalReduction>1</mechanicalReduction>
+      </actuator>
+    </transmission>
+    <transmission name="right_wheel_tran">
+      <type>transmission_interface/SimpleTransmission</type>
+      <joint name="right_wheel_joint">
+	<hardwareInterface>EffortJointInterface</hardwareInterface>
+      </joint>
+      <actuator name="right_wheel_motor">
+	<hardwareInterface>EffortJointInterface</hardwareInterface>
+	<mechanicalReduction>1</mechanicalReduction>
+      </actuator>
+    </transmission>
      <gazebo reference="base_link">
       <material>Gazebo/White</material>

Commit message: camera added to urdf, not working in gazebo

File: urdf/mr_base_macro.xacro (robot description, xacro)
@@ -190,4 +190,66 @@
       </sensor>
     </gazebo>
+    <!--Camera sensor -->
+ <link name="camera_frame">
+      <inertial>
+          <inertia ixx="1.0" ixy="0.0" ixz="0.0" iyy="1.0" iyz="0.0" izz="1.0"/>
+        <mass value="0.1" />
+        <origin xyz="0 0 0" />
+      </inertial>
+      <visual>
+        <geometry>
+		<cylinder length="0.01" radius="0.005"/>
+        </geometry>
+        <material name="White"/>
+        <origin rpy="0 ${-M_PI_2} 0" xyz="0 0 0"/>
+      </visual>
+      <collision>
+        <geometry>
+		<cylinder length="0.01" radius="0.005"/>
+        </geometry>
+        <origin rpy="0 ${-M_PI_2} 0" xyz="0 0 0"/>
+      </collision>
+    </link>
+    <joint name="camera_joint" type="fixed">
+      <parent link="base_link"/>
+      <child link="camera_frame"/>
+      <origin rpy="0 0 0" xyz="0.11 0.0 -0.01"/>
+    </joint>
+    <gazebo reference="sensor">
+    <sensor type="camera" name="camera1">
+      <update_rate>30.0</update_rate>
+      <camera name="head">
+        <horizontal_fov>1.3962634</horizontal_fov>
+        <image>
+          <width>800</width>
+          <height>600</height>
+          <format>R8G8B8</format>
+        </image>
+        <clip>
+          <near>0.02</near>
+          <far>300</far>
+        </clip>
+        <noise>
+          <type>gaussian</type>
+          <mean>0.0</mean>
+          <stddev>0.007</stddev>
+        </noise>
+      </camera>
+      <plugin name="camera_controller" filename="libgazebo_ros_camera.so">
+        <alwaysOn>true</alwaysOn>
+        <updateRate>0.0</updateRate>
+        <cameraName>/camera</cameraName>
+        <imageTopicName>image_raw</imageTopicName>
+        <cameraInfoTopicName>camera_info</cameraInfoTopicName>
+        <frameName>camera_frame</frameName>
+        <hackBaseline>0.07</hackBaseline>
+        <distortionK1>0.0</distortionK1>
+        <distortionK2>0.0</distortionK2>
+        <distortionK3>0.0</distortionK3>
+        <distortionT1>0.0</distortionT1>
+        <distortionT2>0.0</distortionT2>
+      </plugin>
+    </sensor>
+  </gazebo>
     <!-- Differential drive controller  -->
   <gazebo>

Commit message: Planner parameters tuned to better fit our robot model

File: urdf/mr_base_macro.xacro (robot description, xacro)
@@ -215,4 +215,5 @@
       <child link="camera_frame"/>
       <origin rpy="0 0 0" xyz="0.11 0.0 -0.01"/>
+      <!-- <origin rpy="0 0 0" xyz="0.12 0.0 -0.01"/>  -->
     </joint>
     <gazebo reference="camera_frame">

Commit message: Aruco properly working in simulation

File: urdf/mr_base_macro.xacro (robot description, xacro)
@@ -191,5 +191,5 @@
     </gazebo>
     <!--Camera sensor -->
- <link name="camera_frame">
+ <link name="camera_link">
       <inertial>
           <inertia ixx="1.0" ixy="0.0" ixz="0.0" iyy="1.0" iyz="0.0" izz="1.0"/>
@@ -213,9 +213,9 @@
     <joint name="camera_joint" type="fixed">
       <parent link="base_link"/>
-      <child link="camera_frame"/>
-      <origin rpy="0 0 0" xyz="0.11 0.0 -0.01"/>
+      <child link="camera_link"/>
+      <origin rpy="${M_PI} 0 0" xyz="0.11 0.0 -0.01"/>
       <!-- <origin rpy="0 0 0" xyz="0.12 0.0 -0.01"/>  -->
     </joint>
-    <gazebo reference="camera_frame">
+    <gazebo reference="camera_link">
     <sensor type="camera" name="camera1">
       <update_rate>30.0</update_rate>
@@ -243,5 +243,5 @@
         <imageTopicName>image_raw</imageTopicName>
         <cameraInfoTopicName>camera_info</cameraInfoTopicName>
-        <frameName>camera_frame</frameName>
+        <frameName>camera_link</frameName>
         <hackBaseline>0.07</hackBaseline>
         <distortionK1>0.0</distortionK1>

Commit message: Rectified laser orientation in URDF file

File: urdf/mr_base_macro.xacro (robot description, xacro)
@@ -153,5 +153,5 @@
       <parent link="base_link"/>
       <child link="laser"/>
-      <origin rpy="0 0 0" xyz="0.0 0.0 0.155"/>
+      <origin rpy="0 0 ${M_PI}" xyz="0.0 0.0 0.155"/>
     </joint>
     <gazebo reference="laser">

Commit message: Mo vedi che funge

File: urdf/mr_base_macro.xacro (robot description, xacro)
@@ -42,4 +42,6 @@
       </collision>
     </link>
+    <link name="center_link">
+    </link>
     <link name="left_wheel_link">
       <visual>
@@ -87,7 +89,12 @@
     </link>
     <joint name="base_footprint_joint" type="fixed">
-      <parent link="base_footprint"/>
+      <parent link="base_link"/>
+      <child link="base_footprint"/>
+      <origin rpy="0 0 0" xyz="0.0 0.0 -0.059"/>
+    </joint>
+    <joint name="center_joint" type="fixed">
+      <parent link="center_link"/>
       <child link="base_link"/>
-      <origin rpy="0 0 0" xyz="0.0 0.0 0.059"/>
+      <origin rpy="0 0 0" xyz="-0.04025 0.0 0.0"/>
     </joint>
     <joint name="left_wheel_joint" type="continuous">
@@ -260,5 +267,5 @@
       <publishWheelTF>false</publishWheelTF>
       <robotNamespace>/</robotNamespace>
-      <publishTf>1</publishTf>
+      <publishTf>0</publishTf>
       <publishWheelJointState>false</publishWheelJointState>
       <alwaysOn>true</alwaysOn>
@@ -274,5 +281,5 @@
       <odometryFrame>odom</odometryFrame>
       <odometryTopic>odom</odometryTopic>
-      <robotBaseFrame>base_link_gazebo</robotBaseFrame>
+      <robotBaseFrame>base_link</robotBaseFrame>
     </plugin>
   </gazebo>

Commit message: LIDAR rotation fixed

File: urdf/mr_base_macro.xacro (robot description, xacro)
@@ -160,5 +160,5 @@
       <parent link="base_link"/>
       <child link="laser"/>
-      <origin rpy="0 0 ${M_PI}" xyz="0.0 0.0 0.155"/>
+      <origin rpy="0 ${M_PI} 0" xyz="0.0 0.0 0.155"/>
     </joint>
     <gazebo reference="laser">

Commit message: link camera fixed

File: urdf/mr_base_macro.xacro (robot description, xacro)
@@ -147,5 +147,5 @@
         </geometry>
         <material name="White"/>
-        <origin rpy="0 0 ${-M_PI_2}" xyz="0.0 0.0 -0.031"/>
+        <origin rpy="0 ${M_PI} ${M_PI_2}" xyz="0.0 0.0 0.031"/>
       </visual>
       <collision>
@@ -154,5 +154,5 @@
           <cylinder length="0.04" radius="0.037" />
         </geometry>
-        <origin rpy="0 0 0" xyz="0.0 0.0 -0.031"/>
+        <origin rpy="0 0 0" xyz="0.0 0.0 0.031"/>
       </collision>
     </link>
